File: PCB_DESIGN/devboard.kicad_pcb (KiCad board)
At the start: 2 copper layers, 21 x 51 mm, 33 parts, among them J1 USB_C_Receptacle_USB2.0_14P, J2 Conn_01x20, J3 Conn_01x20, J4 Conn_01x03, SW1 SW_Push, U1 RP2040, U2 MCP1700x-330xxTT, U4 W25Q16JVUXIQ TR, Y1 12 MHz

Commit message: working on custom silkscreen
Parts:
- added G***: LOGO, LOGO, F.Cu at (153.8, 127.2)
- added G***: LOGO, LOGO, B.Cu at (153.3, 122.1)
Connections:
- net /USB_DN renamed USB_D-
- net /USB_DP renamed USB_D+
Other:
- board text added: "@KaiPereira"

Commit message: added silkscreen
Parts:
- added G***: LOGO, LOGO, F.Cu at (150.6, 98.6)
- added G***: LOGO, LOGO, B.Cu at (153.4, 98.3)
Other:
- board text added: "HTN!"
- board text added: "kaipereira.com"
